File: PCB/heidi-keyboard/side.kicad_sch (KiCad schematic)
At the start: 65 parts, among them J1 USB_C_Receptacle_USB2.0_14P, J3 AudioJack4, SW1 SW_Push, SW11 SW_Push, SW13 SW_Push, SW14 SW_Push, SW15 SW_Push, SW16 SW_Push, SW17 SW_Push, SW18 SW_Push, SW25 SW_Push, SW26 SW_Push, SW27 SW_Push, SW28 SW_Push, SW29 SW_Push, SW3 SW_Push, SW30 SW_Push, SW37 SW_Push, SW38 SW_Push, SW39 SW_Push, SW40 SW_Push, SW41 SW_Push, SW42 SW_Push, SW49 SW_Push, SW5 SW_Push, SW50 SW_Push, SW51 SW_Push, SW52 SW_Push, SW53 SW_Push, SW54 SW_Push, SW7 SW_Push, SW9 SW_Push

Commit message: aaaaaaaaaaaaaaaa
Parts:
- added D61: LED, symbol Device:LED
- added R2: R, symbol Device:R
- added SW61: RotaryEncoder, symbol Device:RotaryEncoder
Connections:
- net 3V3: now also R2.2; no longer A1.36 (3V3), J3.S
- net GND: now also D61.1 (K), SW61.C
- net GPIO13: now reaches A1.17 (GPIO13)
- net GPIO13: now also SW61.A
- net GPIO14: now reaches A1.19 (GPIO14)
- net GPIO14: now also SW61.B
- net VBUD: now reaches J1.A4 (VBUS), J1.A9 (VBUS), J1.B4 (VBUS), J1.B9 (VBUS)
- net VBUD: no longer A1.40 (VBUS)
- new net: D61.2 (A), R2.1
- new net VBUS: A1.40 (VBUS), J3.S

Commit message: aaaaaaaaaaaa
Parts:
- removed D59: D, symbol Device:D
- removed D61: LED, symbol Device:LED
- removed R2: R, symbol Device:R
- removed SW49: SW_Push, symbol Switch:SW_Push
