File: PCB/heidi-keyboard/heidi-keyboard.kicad_sch (KiCad schematic)
At the start: 0 parts

Commit message: aaaaaaaaaaaaaaaaa
Other:
- sheet right: file side.kicad_sch -> not_side.kicad_sch
Changed lines of the file:
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@@
 			)
 		)
-		(property "Sheetfile" "side.kicad_sch"
+		(property "Sheetfile" "not_side.kicad_sch"
 			(at 76.2 64.0846 0)
 			(effects
@@
 			(project "heidi-keyboard"
 				(path "/fac4024f-04d0-49da-b501-a68e9856b84b"
-					(page "4")
+					(page "3")
 				)
 			)
