File: PCB/heidi-keyboard/heidi-keyboard.kicad_pcb (KiCad board)
At the start: 2 copper layers, 168.5 x 121.2 mm, 33 parts

Commit message: aaaaaaaaaaaaaaaaaaaaaaaaaaaaaaaaaaaaaa
Parts:
- removed the REF** at (73.9, 82.7)
- removed the REF** at (66.0, 45.5)
- added REF**: USB_C_Receptacle_GCT_USB4105-xx-A_16P_TopMnt_Horizontal, Connector_USB:USB_C_Receptacle_GCT_USB4105-xx-A_16P_TopMnt_Horizontal, F.Cu at (57.5, 43.5)
- added REF**: D_SOD-123F, Diode_SMD:D_SOD-123F, F.Cu at (184.5, 105.0)
- added REF**: D_SOD-123F, Diode_SMD:D_SOD-123F, F.Cu at (127.5, 93.5)
- added REF**: D_SOD-123F, Diode_SMD:D_SOD-123F, F.Cu at (195.5, 130.5)
- added REF**: D_SOD-123F, Diode_SMD:D_SOD-123F, F.Cu at (108.5, 79.0)
- added REF**: PinSocket_1x03_P2.54mm_Vertical, Connector_PinSocket_2.54mm:PinSocket_1x03_P2.54mm_Vertical, F.Cu at (85.5, 64.5)
- added REF**: LED_2512_6332Metric_Pad1.52x3.35mm_HandSolder, LED_SMD:LED_2512_6332Metric_Pad1.52x3.35mm_HandSolder, F.Cu at (83.5, 48.0)
- added REF**: D_SOD-123F, Diode_SMD:D_SOD-123F, F.Cu at (108.5, 98.5)
- added REF**: PinSocket_1x20_P2.54mm_Vertical, Connector_PinSocket_2.54mm:PinSocket_1x20_P2.54mm_Vertical, F.Cu at (81.0, 62.9)
- added REF**: D_SOD-123F, Diode_SMD:D_SOD-123F, F.Cu at (146.5, 89.0)
- added REF**: D_SOD-123F, Diode_SMD:D_SOD-123F, F.Cu at (146.5, 70.0)
- added REF**: PinSocket_1x15_P2.54mm_Vertical, Connector_PinSocket_2.54mm:PinSocket_1x15_P2.54mm_Vertical, F.Cu at (85.5, 75.5)
- added REF**: R_0805_2012Metric, Resistor_SMD:R_0805_2012Metric, F.Cu at (58.5, 52.0)
- added REF**: D_SOD-123F, Diode_SMD:D_SOD-123F, F.Cu at (108.5, 117.5)
- added REF**: D_SOD-123F, Diode_SMD:D_SOD-123F, F.Cu at (127.5, 112.5)
- added REF**: D_SOD-123F, Diode_SMD:D_SOD-123F, F.Cu at (184.5, 48.0)
- added REF**: D_SOD-123F, Diode_SMD:D_SOD-123F, F.Cu at (176.0, 126.5)
- added REF**: D_SOD-123F, Diode_SMD:D_SOD-123F, F.Cu at (184.5, 86.0)
- added REF**: D_SOD-123F, Diode_SMD:D_SOD-123F, F.Cu at (127.5, 74.5)
- added REF**: PinSocket_1x20_P2.54mm_Vertical, Connector_PinSocket_2.54mm:PinSocket_1x20_P2.54mm_Vertical, F.Cu at (63.0, 63.0)
- added REF**: R_0805_2012Metric, Resistor_SMD:R_0805_2012Metric, F.Cu at (56.5, 52.0)
- added REF**: D_SOD-123F, Diode_SMD:D_SOD-123F, F.Cu at (146.5, 127.0)
- added REF**: D_SOD-123F, Diode_SMD:D_SOD-123F, F.Cu at (184.5, 67.0)
- added REF**: D_SOD-123F, Diode_SMD:D_SOD-123F, F.Cu at (165.5, 103.0)
- added REF**: D_SOD-123F, Diode_SMD:D_SOD-123F, F.Cu at (127.5, 55.5)
- added REF**: D_SOD-123F, Diode_SMD:D_SOD-123F, F.Cu at (165.5, 84.0)
- added REF**: D_SOD-123F, Diode_SMD:D_SOD-123F, F.Cu at (146.5, 51.0)
- added REF**: D_SOD-123F, Diode_SMD:D_SOD-123F, F.Cu at (165.5, 46.0)
- added REF**: R_0805_2012Metric, Resistor_SMD:R_0805_2012Metric, F.Cu at (80.0, 48.5)
- added REF**: D_SOD-123F, Diode_SMD:D_SOD-123F, F.Cu at (203.5, 69.5)
- added REF**: D_SOD-123F, Diode_SMD:D_SOD-123F, F.Cu at (146.5, 108.0)
- added REF**: D_SOD-123F, Diode_SMD:D_SOD-123F, F.Cu at (127.5, 131.5)
- added REF**: D_SOD-123F, Diode_SMD:D_SOD-123F, F.Cu at (108.5, 60.5)
- added REF**: FanPinHeader_1x04_P2.54mm_Vertical, Connector:FanPinHeader_1x04_P2.54mm_Vertical, F.Cu at (75.6, 46.3)
- added REF**: D_SOD-123F, Diode_SMD:D_SOD-123F, F.Cu at (203.5, 107.5)
- added REF**: D_SOD-123F, Diode_SMD:D_SOD-123F, F.Cu at (165.5, 65.0)
- added REF**: D_SOD-123F, Diode_SMD:D_SOD-123F, F.Cu at (203.5, 88.5)
- added REF**: D_SOD-123F, Diode_SMD:D_SOD-123F, F.Cu at (215.5, 138.0)
- added REF**: D_SOD-123F, Diode_SMD:D_SOD-123F, F.Cu at (203.5, 50.5)
- moved REF** 18.5 mm to (64.0, 123.0), turned to 0 degrees
- moved REF** 0.40 mm to (215.9, 113.0)
Routing:
- net (no net): track 0.00 -> 3675.6 mm, vias 0 -> 43
Other:
- board size 168.5 x 121.2 mm -> 173.5 x 122.5 mm
- board text added: "(symbol "LOGO" (pin_names (offset 1.016)) (in_bom yes) (on_board yes) (property "Reference" "#G" (at 0 12.065 0) (effects (font (size 1.27 1.27)) hide) ) (property "Value" "LOGO" (at 0 -12.065 0) (effects (font (size 1.27 1.27)) hide) ) (property "Footprint" "" (at 0 0 0) (effects (font (size 1.27 1.27)) hide) ) (property "Datasheet" "" (at 0 0 0) (effects (font (size 1.27 1.27)) hide) ) (symbol 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"
- board text added: "D+"
- board text added: "D-"
- board text added: "GND"
- board text added: "VBUS"

Commit message: aaaaaaaaaaaaaaaaaaaaaaaaaaaaaaaa
Parts:
- removed the REF** at (85.5, 64.5)
- removed the REF** at (85.5, 75.5)
- added G***: LOGO, heidi-paws:heidi-hug-blahaj.pretty, F.Cu at (77.0, 86.5)
- added G***: LOGO, heidi-paws:we-all-love-heidi.pretty, F.Cu at (97.5, 128.5)
- added G***: LOGO, heidi-paws:heidi-paws.pretty, F.Cu at (57.5, 128.0)
- added G***: LOGO, heidi-paws:heidi-cute.pretty, F.Cu at (158.5, 126.5)
- added REF**: MountingHole_3.2mm_M3_ISO7380, MountingHole:MountingHole_3.2mm_M3_ISO7380, F.Cu at (203.0, 115.0)
- added REF**: MountingHole_3.2mm_M3_ISO7380, MountingHole:MountingHole_3.2mm_M3_ISO7380, F.Cu at (203.5, 28.5)
- added REF**: MountingHole_3.2mm_M3_ISO7380, MountingHole:MountingHole_3.2mm_M3_ISO7380, F.Cu at (84.0, 125.5)
- added REF**: MountingHole_3.2mm_M3_ISO7380, MountingHole:MountingHole_3.2mm_M3_ISO7380, F.Cu at (52.5, 65.5)
- moved REF** 1.05 mm to (64.5, 122.1)
Routing:
- net (no net): track 3675.6 -> 3654.1 mm, vias 43 -> 42
Other:
- board text removed: "(symbol "LOGO" (pin_names (offset 1.016)) (in_bom yes) (on_board yes) (property "Reference" "#G" (at 0 12.065 0) (effects (font (size 1.27 1.27)) hide) ) (property "Value" "LOGO" (at 0 -12.065 0) (effects (font (size 1.27 1.27)) hide) ) (property "Footprint" "" (at 0 0 0) (effects (font (size 1.27 1.27)) hide) ) (property "Datasheet" "" (at 0 0 0) (effects (font (size 1.27 1.27)) hide) ) (symbol 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"

Commit message: aaaaaaaaaaaaaaaa
Parts:
- moved G*** 21.6 mm to (78.7, 123.6)
- moved G*** 15.7 mm to (92.5, 89.1)
- moved G*** 15.7 mm to (113.0, 131.1)
- moved G*** 15.7 mm to (174.0, 129.1)
- moved REF** 15.7 mm to (73.0, 46.1)
- moved REF** 15.7 mm to (221.5, 131.6)
- moved REF** 15.7 mm to (200.0, 107.6)
- moved REF** 15.7 mm to (143.0, 96.1)
- moved REF** 15.7 mm to (211.0, 133.1)
- moved REF** 15.7 mm to (218.5, 117.6)
- moved REF** 15.7 mm to (124.0, 81.6)
- moved REF** 15.7 mm to (99.0, 50.6)
- moved REF** 15.7 mm to (124.0, 101.1)
- moved REF** 15.7 mm to (96.5, 65.5)
- moved REF** 15.7 mm to (190.5, 98.6)
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Routing:
- net (no net): track 3654.1 -> 3643.7 mm

Commit message: aaaaaaaaaaaaaaaaaaaaaaaaaaaaaaaa
Parts:
- added G***: LOGO, heidi-paws:heidi-huh.pretty, F.Cu at (45.5, 126.5)
- added G***: LOGO, heidi-paws:heidi-pf.pretty, F.Cu at (-9.00, 126.5)
- added G***: LOGO, heidi-paws:heidi-yap.pretty, F.Cu at (123.5, 68.0)
- added G***: LOGO, heidi-paws:heidi-paws-right.pretty, F.Cu at (126.6, 130.7)
- added REF**: D_SOD-123F, Diode_SMD:D_SOD-123F, F.Cu at (86.2, 144.6)
- added REF**: CPG135001S30, PCM_marbastlib-choc:SW_choc_v1_HS_CPG135001S30_1u, F.Cu at (96.0, 64.5)
- added REF**: D_SOD-123F, Diode_SMD:D_SOD-123F, F.Cu at (28.7, 80.1)
- added REF**: CPG135001S30, PCM_marbastlib-choc:SW_choc_v1_HS_CPG135001S30_1u, F.Cu at (58.0, 74.0)
- added REF**: D_SOD-123F, Diode_SMD:D_SOD-123F, F.Cu at (37.5, 139.5)
- added REF**: D_SOD-123F, Diode_SMD:D_SOD-123F, F.Cu at (28.7, 99.1)
- added REF**: CPG135001S30, PCM_marbastlib-choc:SW_choc_v1_HS_CPG135001S30_1u, F.Cu at (96.0, 121.5)
- added REF**: mousebites 2mm, PCM_marbastlib-various:mousebites_2.5mm, F.Cu at (149.0, 143.0)
- added REF**: D_SOD-123F, Diode_SMD:D_SOD-123F, F.Cu at (10.2, 82.6)
- added REF**: D_SOD-123F, Diode_SMD:D_SOD-123F, F.Cu at (86.2, 68.6)
- added REF**: D_SOD-123F, Diode_SMD:D_SOD-123F, F.Cu at (105.2, 92.6)
- added REF**: CPG135001S30, PCM_marbastlib-choc:SW_choc_v1_HS_CPG135001S30_1u, F.Cu at (58.0, 93.0)
- added REF**: D_SOD-123F, Diode_SMD:D_SOD-123F, F.Cu at (105.2, 111.6)
- added REF**: CPG135001S30, PCM_marbastlib-choc:SW_choc_v1_HS_CPG135001S30_1u, F.Cu at (96.0, 83.5)
- added REF**: D_SOD-123F, Diode_SMD:D_SOD-123F, F.Cu at (105.2, 73.6)
- added REF**: D_SOD-123F, Diode_SMD:D_SOD-123F, F.Cu at (18.0, 143.5)
- added REF**: CPG135001S30, PCM_marbastlib-choc:SW_choc_v1_HS_CPG135001S30_1u, F.Cu at (77.0, 78.5)
- added REF**: CPG135001S30, PCM_marbastlib-choc:SW_choc_v1_HS_CPG135001S30_1u, F.Cu at (28.5, 130.5)
- added REF**: CPG135001S30, PCM_marbastlib-choc:SW_choc_v1_HS_CPG135001S30_1u, F.Cu at (39.0, 69.0)
- added REF**: D_SOD-123F, Diode_SMD:D_SOD-123F, F.Cu at (67.2, 83.1)
- added REF**: CPG135001S30, PCM_marbastlib-choc:SW_choc_v1_HS_CPG135001S30_1u, F.Cu at (8.89, 134.5)
- added REF**: D_SOD-123F, Diode_SMD:D_SOD-123F, F.Cu at (48.2, 116.1)
- added REF**: RotaryEncoder_Alps_EC12E_Vertical_H20mm, Rotary_Encoder:RotaryEncoder_Alps_EC12E_Vertical_H20mm, F.Cu at (121.5, 73.0)
- added REF**: MountingHole_3.2mm_M3_ISO7380, MountingHole:MountingHole_3.2mm_M3_ISO7380, B.Cu at (-8.50, 41.5)
- added REF**: MountingHole_3.2mm_M3_ISO7380, MountingHole:MountingHole_3.2mm_M3_ISO7380, B.Cu at (111.0, 138.5)
- added REF**: CPG135001S30, PCM_marbastlib-choc:SW_choc_v1_HS_CPG135001S30_1u, F.Cu at (1.00, 111.5)
- added REF**: MountingHole_3.2mm_M3_ISO7380, MountingHole:MountingHole_3.2mm_M3_ISO7380, B.Cu at (-8.00, 128.0)
- added REF**: MountingHole_3.2mm_M3_ISO7380, MountingHole:MountingHole_3.2mm_M3_ISO7380, B.Cu at (142.5, 78.5)
- added REF**: CPG135001S30, PCM_marbastlib-choc:SW_choc_v1_HS_CPG135001S30_1u, F.Cu at (77.0, 135.5)
- added REF**: CPG135001S30, PCM_marbastlib-choc:SW_choc_v1_HS_CPG135001S30_1u, F.Cu at (77.0, 59.5)
- added REF**: CPG135001S30, PCM_marbastlib-choc:SW_choc_v1_HS_CPG135001S30_1u, F.Cu at (39.0, 107.0)
- added REF**: CPG135001S30, PCM_marbastlib-choc:SW_choc_v1_HS_CPG135001S30_1u, F.Cu at (77.0, 97.5)
- added REF**: D_SOD-123F, Diode_SMD:D_SOD-123F, F.Cu at (48.2, 59.1)
- added REF**: PinSocket_1x20_P2.54mm_Vertical, Connector_PinSocket_2.54mm:PinSocket_1x20_P2.54mm_Vertical, F.Cu at (113.7, 81.5)
- added REF**: CPG135001S30, PCM_marbastlib-choc:SW_choc_v1_HS_CPG135001S30_1u, F.Cu at (-11.0, 142.0)
- added REF**: D_SOD-123F, Diode_SMD:D_SOD-123F, F.Cu at (105.2, 130.6)
- added REF**: D_SOD-123F, Diode_SMD:D_SOD-123F, F.Cu at (48.2, 78.1)
- added REF**: D_SOD-123F, Diode_SMD:D_SOD-123F, F.Cu at (67.2, 140.1)
- added REF**: D_SOD-123F, Diode_SMD:D_SOD-123F, F.Cu at (10.2, 120.6)
- added REF**: D_SOD-123F, Diode_SMD:D_SOD-123F, F.Cu at (67.2, 102.1)
- added REF**: CPG135001S30, PCM_marbastlib-choc:SW_choc_v1_HS_CPG135001S30_1u, F.Cu at (1.00, 54.5)
- added REF**: D_SOD-123F, Diode_SMD:D_SOD-123F, F.Cu at (-2.00, 151.0)
- added REF**: D_SOD-123F, Diode_SMD:D_SOD-123F, F.Cu at (28.7, 61.1)
- added REF**: MJ-4PP-9, PCM_marbastlib-xp-various:CON_MJ-4PP-9, F.Cu at (-20.9, 126.0)
- added REF**: CPG135001S30, PCM_marbastlib-choc:SW_choc_v1_HS_CPG135001S30_1u, F.Cu at (58.0, 131.0)
- added REF**: mousebites 2mm, PCM_marbastlib-various:mousebites_2.5mm, F.Cu at (149.0, 96.0)
- added REF**: D_SOD-123F, Diode_SMD:D_SOD-123F, F.Cu at (86.2, 106.6)
- added REF**: CPG135001S30, PCM_marbastlib-choc:SW_choc_v1_HS_CPG135001S30_1u, F.Cu at (20.0, 109.0)
- added REF**: CPG135001S30, PCM_marbastlib-choc:SW_choc_v1_HS_CPG135001S30_1u, F.Cu at (96.0, 102.5)
- added REF**: D_SOD-123F, Diode_SMD:D_SOD-123F, F.Cu at (28.7, 118.1)
- added REF**: CPG135001S30, PCM_marbastlib-choc:SW_choc_v1_HS_CPG135001S30_1u, F.Cu at (39.0, 88.0)
- added REF**: CPG135001S30, PCM_marbastlib-choc:SW_choc_v1_HS_CPG135001S30_1u, F.Cu at (58.0, 55.0)
- added REF**: D_SOD-123F, Diode_SMD:D_SOD-123F, F.Cu at (67.2, 121.1)
- added REF**: D_SOD-123F, Diode_SMD:D_SOD-123F, F.Cu at (86.2, 125.6)
- added REF**: D_SOD-123F, Diode_SMD:D_SOD-123F, F.Cu at (10.2, 101.6)
- added REF**: D_SOD-123F, Diode_SMD:D_SOD-123F, F.Cu at (48.2, 97.1)
- added REF**: CPG135001S30, PCM_marbastlib-choc:SW_choc_v1_HS_CPG135001S30_1u, F.Cu at (20.0, 90.0)
- added REF**: D_SOD-123F, Diode_SMD:D_SOD-123F, F.Cu at (67.2, 64.1)
- added REF**: CPG135001S30, PCM_marbastlib-choc:SW_choc_v1_HS_CPG135001S30_1u, F.Cu at (58.0, 112.0)
- added REF**: CPG135001S30, PCM_marbastlib-choc:SW_choc_v1_HS_CPG135001S30_1u, F.Cu at (1.00, 73.5)
- added REF**: CPG135001S30, PCM_marbastlib-choc:SW_choc_v1_HS_CPG135001S30_1u, F.Cu at (39.0, 50.0)
- added REF**: mousebites 2mm, PCM_marbastlib-various:mousebites_2.5mm, F.Cu at (149.0, 62.5)
- added REF**: CPG135001S30, PCM_marbastlib-choc:SW_choc_v1_HS_CPG135001S30_1u, F.Cu at (77.0, 116.5)
- added REF**: D_SOD-123F, Diode_SMD:D_SOD-123F, F.Cu at (10.2, 63.6)
- added REF**: PinSocket_1x20_P2.54mm_Vertical, Connector_PinSocket_2.54mm:PinSocket_1x20_P2.54mm_Vertical, F.Cu at (131.7, 81.6)
- added REF**: D_SOD-123F, Diode_SMD:D_SOD-123F, F.Cu at (86.2, 87.6)
- added REF**: CPG135001S30, PCM_marbastlib-choc:SW_choc_v1_HS_CPG135001S30_1u, F.Cu at (20.0, 52.0)
- added REF**: CPG135001S30, PCM_marbastlib-choc:SW_choc_v1_HS_CPG135001S30_1u, F.Cu at (1.00, 92.5)
- added REF**: CPG135001S30, PCM_marbastlib-choc:SW_choc_v1_HS_CPG135001S30_1u, F.Cu at (20.0, 71.0)
- moved G*** 89.0 mm to (167.2, 133.0)
- moved G*** 85.6 mm to (259.0, 139.5)
- moved REF** 85.6 mm to (294.5, 73.5)
- moved REF** 85.6 mm to (266.0, 59.0)
- moved REF** 85.6 mm to (304.0, 82.5)
- moved REF** 85.6 mm to (294.5, 111.5)
- moved REF** 85.6 mm to (304.0, 120.5)
- moved REF** 85.6 mm to (266.0, 78.0)
- moved REF** 85.6 mm to (304.0, 101.5)
- moved REF** 85.6 mm to (316.0, 151.0)
- moved REF** 85.6 mm to (316.4, 126.0)
- moved REF** 85.6 mm to (275.5, 52.0)
- moved REF** 85.6 mm to (256.5, 50.0)
- moved REF** 85.6 mm to (304.0, 63.5)
- moved REF** 85.6 mm to (306.5, 142.0)
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Routing:
- net (no net): track 3643.7 -> 6645.9 mm, vias 42 -> 80
Other:
- board size 173.5 x 122.5 mm -> 349.5 x 122.5 mm
- board text added: "${REFERENCE}"
