File: PCB/heidi-keyboard/_autosave-heidi-keyboard.kicad_pcb (KiCad board)
At the start: 2 copper layers, 349.5 x 122.5 mm, 184 parts

Commit message: aaaaaaaaaaaaaaaaaaa
Parts:
- added REF**: LED_0805_2012Metric, LED_SMD:LED_0805_2012Metric, F.Cu at (218.5, 54.8)
- added REF**: LED_0805_2012Metric, LED_SMD:LED_0805_2012Metric, F.Cu at (237.5, 88.3)
- added REF**: LED_0805_2012Metric, LED_SMD:LED_0805_2012Metric, F.Cu at (294.5, 87.8)
- added REF**: LED_0805_2012Metric, LED_SMD:LED_0805_2012Metric, F.Cu at (275.5, 85.3)
- added REF**: LED_0805_2012Metric, LED_SMD:LED_0805_2012Metric, F.Cu at (256.5, 45.3)
- added REF**: LED_0805_2012Metric, LED_SMD:LED_0805_2012Metric, F.Cu at (218.5, 111.8)
- added REF**: LED_0805_2012Metric, LED_SMD:LED_0805_2012Metric, F.Cu at (218.5, 73.8)
- added REF**: LED_0805_2012Metric, LED_SMD:LED_0805_2012Metric, F.Cu at (256.5, 102.3)
- added REF**: LED_0805_2012Metric, LED_SMD:LED_0805_2012Metric, F.Cu at (275.5, 47.3)
- added REF**: LED_0805_2012Metric, LED_SMD:LED_0805_2012Metric, F.Cu at (275.5, 104.3)
- added REF**: LED_0805_2012Metric, LED_SMD:LED_0805_2012Metric, F.Cu at (286.6, 129.8)
- added REF**: LED_0805_2012Metric, LED_SMD:LED_0805_2012Metric, F.Cu at (199.5, 59.8)
- added REF**: LED_0805_2012Metric, LED_SMD:LED_0805_2012Metric, F.Cu at (199.5, 78.8)
- added REF**: R_0805_2012Metric, Resistor_SMD:R_0805_2012Metric, F.Cu at (199.5, 54.0)
- added REF**: LED_0805_2012Metric, LED_SMD:LED_0805_2012Metric, F.Cu at (199.5, 116.8)
- added REF**: LED_0805_2012Metric, LED_SMD:LED_0805_2012Metric, F.Cu at (218.5, 130.8)
- added REF**: R_0805_2012Metric, Resistor_SMD:R_0805_2012Metric, F.Cu at (256.5, 39.5)
- added REF**: R_0805_2012Metric, Resistor_SMD:R_0805_2012Metric, F.Cu at (294.5, 44.0)
- added REF**: LED_0805_2012Metric, LED_SMD:LED_0805_2012Metric, F.Cu at (199.5, 97.8)
- added REF**: R_0805_2012Metric, Resistor_SMD:R_0805_2012Metric, F.Cu at (275.5, 41.5)
- added REF**: LED_0805_2012Metric, LED_SMD:LED_0805_2012Metric, F.Cu at (256.5, 83.3)
- added REF**: LED_0805_2012Metric, LED_SMD:LED_0805_2012Metric, F.Cu at (294.5, 68.8)
- added REF**: R_0805_2012Metric, Resistor_SMD:R_0805_2012Metric, F.Cu at (218.5, 49.0)
- added REF**: LED_0805_2012Metric, LED_SMD:LED_0805_2012Metric, F.Cu at (218.5, 92.8)
- added REF**: LED_0805_2012Metric, LED_SMD:LED_0805_2012Metric, F.Cu at (267.0, 125.8)
- added REF**: LED_0805_2012Metric, LED_SMD:LED_0805_2012Metric, F.Cu at (237.5, 69.3)
- added REF**: LED_0805_2012Metric, LED_SMD:LED_0805_2012Metric, F.Cu at (256.5, 64.3)
- added REF**: R_0805_2012Metric, Resistor_SMD:R_0805_2012Metric, F.Cu at (237.5, 44.5)
- added REF**: LED_0805_2012Metric, LED_SMD:LED_0805_2012Metric, F.Cu at (237.5, 107.3)
- added REF**: LED_0805_2012Metric, LED_SMD:LED_0805_2012Metric, F.Cu at (275.5, 66.3)
- added REF**: LED_0805_2012Metric, LED_SMD:LED_0805_2012Metric, F.Cu at (237.5, 126.3)
- added REF**: LED_0805_2012Metric, LED_SMD:LED_0805_2012Metric, F.Cu at (294.5, 106.8)
- added REF**: LED_0805_2012Metric, LED_SMD:LED_0805_2012Metric, F.Cu at (294.5, 49.8)
- added REF**: LED_0805_2012Metric, LED_SMD:LED_0805_2012Metric, F.Cu at (306.5, 137.3)
- added REF**: LED_0805_2012Metric, LED_SMD:LED_0805_2012Metric, F.Cu at (237.5, 50.3)
Routing:
- net (no net): track 8103.0 -> 8484.3 mm, vias 156 -> 169
Other:
- board text added: "← 40Ω"
